File: board/RISKYMSX2.kicad_sch (KiCad schematic)
At the start: 47 parts, among them CN1 MSX_CART, IC1 LM1117MPX-3.3, J1 Conn_01x02, J2 Conn_01x02, J3 Conn_01x02, J4 USB_1, U1 CH32V467VET6, U2 MCP6001-OT, Y1 25Mhz

Commit message: terminal improvements
Parts:
- removed C14: 100nF, Capacitor_SMD:C_0603_1608Metric_Pad1.08x0.95mm_HandSolder, symbol Device:C
- removed C4: 100nF, Capacitor_SMD:C_0603_1608Metric_Pad1.08x0.95mm_HandSolder, symbol Device:C_Small
- removed R2: 10K, Resistor_SMD:R_0603_1608Metric_Pad0.98x0.95mm_HandSolder, symbol Device:R
- C1, C10, C11, C12, C13, C21, C28, C7, C8, C9: value 100nF -> 100n
- C15, C16, C17, C18, C19, C2: value 10uF -> 10u
- C20, C3: value 1uF -> 1u
- C22, C24: value 15p -> 18p
- C23, C27: value 1nF -> 1n
- C25, C26: value 4.7uF -> 4.7u
- C5, C6: value 2.2uF -> 2.2u
- IC1: value LM1117MPX-3.3 -> LM1117-3.3
- Y1: footprint Crystal:Crystal_SMD_7050-4Pin_7.0x5.0mm -> Crystal:Crystal_HC49-4H_Vertical
Connections:
- net +3.3V: now also U1.22 (VDDA)
- net NRST: no longer names the net of U1.14 (~{NRST})
- no-connect marks 33 -> 34
