File: board/RISKYMSX2.kicad_pcb (KiCad board)
At the start: 4 copper layers, 71.9 x 55.5 mm, 48 parts, among them CN1 MSX_CART, IC1 LM1117 3.3V, J1 Conn_01x02, J2 Conn_01x02, J3 Conn_01x02, J4 USB_1, U1 CH32V467VET6, U2 MCP6001-OT, Y1 25Mhz

Commit message: terminal improvements
Parts:
- removed C14, C4: 100n, Capacitor_SMD:C_0603_1608Metric_Pad1.08x0.95mm_HandSolder
- removed R2: 10K, Resistor_SMD:R_0603_1608Metric_Pad0.98x0.95mm_HandSolder
- C11, C17, C28: moved to B.Cu
- C19: value 10uF -> 10u
- C22, C24: value 15p -> 18p; moved to B.Cu
- IC1: value LM1117 3.3V -> LM1117-3.3
- Y1: footprint Crystal:Crystal_SMD_7050-4Pin_7.0x5.0mm -> Crystal:Crystal_HC49-4H_Vertical
- moved C17 6.40 mm to (156.0, 103.3)
- moved C28 6.34 mm to (154.6, 103.3)
- moved C11 4.80 mm to (155.5, 99.1)
- moved Y1 3.21 mm to (164.6, 99.0)
- moved C22 1.27 mm to (164.6, 106.5)
- moved C24 0.89 mm to (164.6, 96.3)
Connections:
- U1 pad 14: /NRST -> unconnected-(U1-~{NRST}-Pad14)
- U1 pad 22: Net-(U1-VDDA) -> +3.3V
Routing:
- net /IORQ: track 50.3 -> 55.1 mm
- net /NRST: track 3.80 -> 0.00 mm, vias 1 -> 0
- net /BDIR: track 51.6 -> 55.0 mm
- net GND: track 52.3 -> 49.1 mm, vias 33 -> 31
- net /SWDIO: track 7.49 -> 4.80 mm
- net /A8: track 38.9 -> 41.5 mm
- net /D6: track 41.7 -> 39.6 mm
- net +3.3V: track 39.7 -> 41.6 mm, vias 20 -> 19
- net Net-(U1-VDDA): track 1.89 -> 0.00 mm, vias 1 -> 0
- net /A3: track 27.8 -> 29.5 mm
- net /D4: track 39.9 -> 38.3 mm
- net Net-(U1-OSC_OUT): track 10.7 -> 9.41 mm
- net Net-(U1-OSC_IN): track 11.0 -> 10.2 mm
- net /D2: track 43.4 -> 44.1 mm
- net /SLOTINT: track 49.5 -> 48.8 mm
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
Commit message: New PCB
Parts:
- C22, C24: moved to F.Cu
- moved C24 5.25 mm to (169.1, 99.0), turned to 180 degrees
- moved C22 5.20 mm to (169.1, 104.0), turned to 180 degrees
- moved J1 0.63 mm to (141.3, 112.5)
Routing:
- net /IORQ: track 55.1 -> 59.8 mm
- net /BDIR: track 55.0 -> 58.9 mm
- net Net-(U1-OSC_IN): track 10.2 -> 12.6 mm
- net Net-(U1-OSC_OUT): track 9.41 -> 11.4 mm
- net /MREQ: track 28.0 -> 27.1 mm
- net /~{RESET}: track 25.6 -> 24.7 mm
- net /WAIT: track 34.4 -> 33.8 mm
- net GND: vias 31 -> 53
- added copper zone on B.Cu, net GND
- added copper zone on F.Cu, net GND
Other:
- board text added: "Rev 0.2 PROTOTYPE"
- board text removed: "Rev 0.1 PROTOTYPE"
